File: kicad/drink-me-usb-c/drink-me.kicad_pcb (KiCad board)
At the start: 2 copper layers, 94 x 29 mm, 22 parts, among them J0 AVR-ISP-6, J1 USB4105_REVA, K0 KEYSW, K1 KEYSW, K2 KEYSW, K3 KEYSW, SW1 RESET, U1 32U2-AU, Y1 16Mhz

Commit message: Use HRO TYPE-C-31-M-12 USB-C connector. Add bill of materials. Add printed back part without rest, including tolerance adjustments.
Parts:
- J1: value USB4105_REVA -> HRO-TYPE-C-31-M-12; footprint SnapEDA:GCT_USB4105_REVA -> Type-C:HRO-TYPE-C-31-M-12-Assembly
- moved J1 2.80 mm to (74.0, 64.0)
- turned R5 to 180 degrees
Connections:
- R5 pad 1: Net-(J1-PadA5) -> GND
- R5 pad 2: GND -> Net-(J1-Pad4)
- R6 pad 2: Net-(J1-PadB5) -> Net-(J1-Pad10)
Routing:
- net Net-(J1-Pad10): track 0.00 -> 14.9 mm, vias 0 -> 2
- net Net-(J1-PadB5): track 14.8 -> 0.00 mm, vias 2 -> 0
- net Net-(J1-Pad4): track 0.00 -> 14.7 mm, vias 0 -> 2
- net Net-(J1-PadA5): track 14.6 -> 0.00 mm, vias 2 -> 0
- net GND: track 161.3 -> 153.7 mm
- net (no net): track 0.00 -> 6.00 mm
Other:
- board text added: "JLCJLCJLCJLC"
- board text added: "v1.0"
- board text removed: "v0.2"
