File: kicad/drink-me-usb-micro/drink-me.sch (KiCad schematic (older format))
At the start: 20 parts, among them J0 AVR-ISP-6, J1 USB_mini_micro_B, K0 KEYSW, K1 KEYSW, K2 KEYSW, K3 KEYSW, SW1 RESET, U1 32U2-AU, Y1 16Mhz

Commit message: Use HRO TYPE-C-31-M-12 USB-C connector. Add bill of materials. Add printed back part without rest, including tolerance adjustments.
Parts:
- C1, C2: BomReferenceDigiKey (none) -> 311-1103-1-ND; ComponentStencilOpenSCAD (none) -> csquare([2, 1.2]);
- C3, C4: BomReferenceDigiKey (none) -> 311-1361-1-ND; ComponentStencilOpenSCAD (none) -> csquare([2, 1.2]);
- C5: BomReferenceDigiKey (none) -> 311-1371-1-ND; ComponentStencilOpenSCAD (none) -> csquare([2, 1.2]);
- C8: BomReferenceDigiKey (none) -> 311-1909-1-ND; ComponentStencilOpenSCAD (none) -> csquare([2, 1.2]);
- F1: BomReferenceDigiKey (none) -> 0ZCJ0050AF2E; ComponentStencilOpenSCAD (none) -> csquare([3.2, 1.6]);
- J1: BomReferenceDigiKey (none) -> H125718CT-ND; ComponentStencilOpenSCAD (none) -> csquare([9.6, 7.6]);
- K0, K1, K2, K3: ComponentStencilOpenSCAD (none) -> translate([0.635, -3.81]) csquare([14.5, 5.9]);
- R1, R2: BomReferenceDigiKey (none) -> CR0805-JW-103ELFCT-ND; ComponentStencilOpenSCAD (none) -> csquare([2, 1.2]);
- R3, R4: BomReferenceDigiKey (none) -> 118-CR0805-JW-220ELFCT-ND; ComponentStencilOpenSCAD (none) -> csquare([2, 1.2]);
- SW1: BomReferenceDigiKey (none) -> EG5470CT-ND; ComponentStencilOpenSCAD (none) -> csquare([6.6, 5.1]);
- U1: BomReferenceDigiKey (none) -> ATMEGA32U2-AURCT-ND; ComponentStencilOpenSCAD (none) -> csquare([9.2, 9.2]);
- Y1: BomReferenceDigiKey (none) -> SER3686CT-ND; ComponentStencilOpenSCAD (none) -> csquare([3.2, 2.5]);
