File: kicad/drink-me-usb-mini/drink-me.kicad_pcb (KiCad board)
At the start: 2 copper layers, 94 x 29 mm, 20 parts, among them J0 AVR-ISP-6, J1 USB_mini_micro_B, K0 KEYSW, K1 KEYSW, K2 KEYSW, K3 KEYSW, SW1 RESET, U1 32U2-AU, Y1 16Mhz

Commit message: Use HRO TYPE-C-31-M-12 USB-C connector. Add bill of materials. Add printed back part without rest, including tolerance adjustments.
Other:
- board text added: "JLCJLCJLCJLC"
- board text added: "v1.0"
- board text removed: "v0.2"
